File: hardware/PiPiNRF.kicad_sch (KiCad schematic)
At the start: 2 parts, among them U2 NRF24L01_Breakout

Commit message: Working Software
Parts:
- A1: footprint PiPico:RaspberryPi_Pico_Common -> Module_RaspberryPi_Pico:RaspberryPi_Pico_Common
Changed lines of the file:
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@@
 			)
 		)
-		(property "Footprint" "PiPico:RaspberryPi_Pico_Common"
+		(property "Footprint" "Module_RaspberryPi_Pico:RaspberryPi_Pico_Common"
 			(at 85.09 43.18 0)
 			(effects
